Commit message: gripper not working properly

File: src/flexiv_ros2/flexiv_description/urdf/rizon.urdf.xacro (robot description, xacro)
@@ -7,4 +7,6 @@
   <!-- import main macro -->
   <xacro:include filename="$(find flexiv_description)/urdf/rizon_macro.xacro"/>
+  <!-- Import gripper-->
+  <xacro:include filename="$(find flexiv_description)/urdf/grav.urdf.xacro"/>
   <!-- parameters -->
   <xacro:arg name="prefix" default="" />
@@ -25,4 +27,13 @@
     initial_positions="${xacro.load_yaml(initial_positions_file)}">
   </xacro:rizon_robot>
+  <!-- Include the gripper macro with the appropriate prefix
+  <xacro:gripper prefix="$(arg prefix)"/>
+    <xacro:gripper prefix="gripper_"/>
+    <joint name="gripper_base_joint" type="fixed">
+      <origin xyz="0 0 0" rpy="0 0 0"/>
+      <parent link="flange"/>
+      <child link="gripper_base_link"/>
+    </joint>
+  -->
   <!-- JointStatePublisher publishes joint state information for the model.
          In future versions of Gazebo, replace 'ignition-gazebo' with 'gz-sim' and
