Commit message: added gripper

File: src/flexiv_ros2/flexiv_description/urdf/grav.urdf.xacro (robot description, xacro)
@@ -1,7 +1,7 @@
 <?xml version="1.0"?>
 <robot xmlns:xacro="http://www.ros.org/wiki/xacro" name="flexiv_GN01">
-  <xacro:macro name="gripper" params="prefix">
+  <xacro:macro name="gripper" params="gripper_prefix">
     <!-- base link -->
-    <link name="${prefix}base_link">
+    <link name="${gripper_prefix}base_link">
       <inertial>
         <origin rpy="0 0 0" xyz="0 0 0.057"/>
@@ -24,9 +24,9 @@
     </link>
     <!-- left finger links -->
-    <link name="${prefix}left_outer_bar">
-      <inertial>
-        <origin xyz="0 0 0.029" rpy="0 0 0"/>
-        <mass value="0.0001"/>
-        <inertia ixx="0.0000001" ixy="0" ixz="0" iyy="0.0000001" iyz="0" izz="0.0000001"/>
+    <link name="${gripper_prefix}left_outer_bar">
+      <inertial>
+        <origin xyz="0 0 0.029" rpy="0 0 0"/>
+        <mass value="0.01"/> <!-- Adjusted mass -->
+        <inertia ixx="0.00001" ixy="0" ixz="0" iyy="0.00001" iyz="0" izz="0.00001"/> <!-- Adjusted inertia -->
       </inertial>
       <visual>
@@ -38,9 +38,9 @@
       </visual>
     </link>
-    <link name="${prefix}left_inner_bar">
-      <inertial>
-        <origin xyz="0 0 0.029" rpy="0 0 0"/>
-        <mass value="0.0001"/>
-        <inertia ixx="0.0000001" ixy="0" ixz="0" iyy="0.0000001" iyz="0" izz="0.0000001"/>
+    <link name="${gripper_prefix}left_inner_bar">
+      <inertial>
+        <origin xyz="0 0 0.029" rpy="0 0 0"/>
+        <mass value="0.01"/> <!-- Adjusted mass -->
+        <inertia ixx="0.00001" ixy="0" ixz="0" iyy="0.00001" iyz="0" izz="0.00001"/> <!-- Adjusted inertia -->
       </inertial>
       <visual>
@@ -52,9 +52,10 @@
       </visual>
     </link>
-    <link name="${prefix}left_finger_mount">
+    <!-- Continue with other links similarly -->
+    <link name="${gripper_prefix}left_finger_mount">
       <inertial>
         <origin xyz="0 0 0" rpy="0 0 0"/>
-        <mass value="0.0001"/>
-        <inertia ixx="0.0000001" ixy="0" ixz="0" iyy="0.0000001" iyz="0" izz="0.0000001"/>
+        <mass value="0.01"/> <!-- Adjusted mass -->
+        <inertia ixx="0.00001" ixy="0" ixz="0" iyy="0.00001" iyz="0" izz="0.00001"/> <!-- Adjusted inertia -->
       </inertial>
       <visual>
@@ -66,9 +67,9 @@
       </visual>
     </link>
-    <link name="${prefix}left_finger_tip">
-      <inertial>
-        <origin rpy="0 0 0" xyz="0 0 0"/>
-        <mass value="0"/>
-        <inertia ixx="0" ixy="0" ixz="0" iyy="0" iyz="0" izz="0"/>
+    <link name="${gripper_prefix}left_finger_tip">
+      <inertial>
+        <origin rpy="0 0 0" xyz="0 0 0"/>
+        <mass value="0.01"/> <!-- Adjusted mass -->
+        <inertia ixx="0.00001" ixy="0" ixz="0" iyy="0.00001" iyz="0" izz="0.00001"/> <!-- Adjusted inertia -->
       </inertial>
       <visual>
@@ -86,9 +87,9 @@
     </link>
     <!-- right finger links -->
-    <link name="${prefix}right_outer_bar">
-      <inertial>
-        <origin xyz="0 0 0.029" rpy="0 0 0"/>
-        <mass value="0.0001"/>
-        <inertia ixx="0.0000001" ixy="0" ixz="0" iyy="0.0000001" iyz="0" izz="0.0000001"/>
+    <link name="${gripper_prefix}right_outer_bar">
+      <inertial>
+        <origin xyz="0 0 0.029" rpy="0 0 0"/>
+        <mass value="0.01"/> <!-- Adjusted mass -->
+        <inertia ixx="0.00001" ixy="0" ixz="0" iyy="0.00001" iyz="0" izz="0.00001"/> <!-- Adjusted inertia -->
       </inertial>
       <visual>
@@ -100,9 +101,9 @@
       </visual>
     </link>
-    <link name="${prefix}right_inner_bar">
-      <inertial>
-        <origin xyz="0 0 0.029" rpy="0 0 0"/>
-        <mass value="0.0001"/>
-        <inertia ixx="0.0000001" ixy="0" ixz="0" iyy="0.0000001" iyz="0" izz="0.0000001"/>
+    <link name="${gripper_prefix}right_inner_bar">
+      <inertial>
+        <origin xyz="0 0 0.029" rpy="0 0 0"/>
+        <mass value="0.01"/> <!-- Adjusted mass -->
+        <inertia ixx="0.00001" ixy="0" ixz="0" iyy="0.00001" iyz="0" izz="0.00001"/> <!-- Adjusted inertia -->
       </inertial>
       <visual>
@@ -114,9 +115,9 @@
       </visual>
     </link>
-    <link name="${prefix}right_finger_mount">
+    <link name="${gripper_prefix}right_finger_mount">
       <inertial>
         <origin xyz="0 0 0" rpy="0 0 0"/>
-        <mass value="0.0001"/>
-        <inertia ixx="0.0000001" ixy="0" ixz="0" iyy="0.0000001" iyz="0" izz="0.0000001"/>
+        <mass value="0.01"/> <!-- Adjusted mass -->
+        <inertia ixx="0.00001" ixy="0" ixz="0" iyy="0.00001" iyz="0" izz="0.00001"/> <!-- Adjusted inertia -->
       </inertial>
       <visual>
@@ -128,9 +129,9 @@
       </visual>
     </link>
-    <link name="${prefix}right_finger_tip">
-      <inertial>
-        <origin rpy="0 0 0" xyz="0 0 0"/>
-        <mass value="0"/>
-        <inertia ixx="0" ixy="0" ixz="0" iyy="0" iyz="0" izz="0"/>
+    <link name="${gripper_prefix}right_finger_tip">
+      <inertial>
+        <origin rpy="0 0 0" xyz="0 0 0"/>
+        <mass value="0.01"/> <!-- Adjusted mass -->
+        <inertia ixx="0.00001" ixy="0" ixz="0" iyy="0.00001" iyz="0" izz="0.00001"/> <!-- Adjusted inertia -->
       </inertial>
       <visual>
@@ -148,131 +149,132 @@
     </link>
     <!-- TCP links -->
-    <link name="${prefix}tcp">
-      <inertial>
-        <origin rpy="0 0 0" xyz="0 0 0"/>
-        <mass value="0"/>
-        <inertia ixx="0" ixy="0" ixz="0" iyy="0" iyz="0" izz="0"/>
-      </inertial>
-    </link>
-    <link name="${prefix}closed_fingers_tcp">
-      <inertial>
-        <origin rpy="0 0 0" xyz="0 0 0"/>
-        <mass value="0"/>
-        <inertia ixx="0" ixy="0" ixz="0" iyy="0" iyz="0" izz="0"/>
-      </inertial>
-    </link>
-    <link name="${prefix}left_finger_tcp">
-      <inertial>
-        <origin rpy="0 0 0" xyz="0 0 0"/>
-        <mass value="0"/>
-        <inertia ixx="0" ixy="0" ixz="0" iyy="0" iyz="0" izz="0"/>
-      </inertial>
-    </link>
-    <link name="${prefix}right_finger_tcp">
-      <inertial>
-        <origin rpy="0 0 0" xyz="0 0 0"/>
-        <mass value="0"/>
-        <inertia ixx="0" ixy="0" ixz="0" iyy="0" iyz="0" izz="0"/>
-      </inertial>
-    </link>
-    <joint name="${prefix}open_fingers_tcp_joint" type="fixed">
+    <link name="${gripper_prefix}tcp">
+      <inertial>
+        <origin rpy="0 0 0" xyz="0 0 0"/>
+        <mass value="0.01"/> <!-- Adjusted mass -->
+        <inertia ixx="0.00001" ixy="0" ixz="0" iyy="0.00001" iyz="0" izz="0.00001"/> <!-- Adjusted inertia -->
+      </inertial>
+    </link>
+    <link name="${gripper_prefix}closed_fingers_tcp">
+      <inertial>
+        <origin rpy="0 0 0" xyz="0 0 0"/>
+        <mass value="0.01"/> <!-- Adjusted mass -->
+        <inertia ixx="0.00001" ixy="0" ixz="0" iyy="0.00001" iyz="0" izz="0.00001"/> <!-- Adjusted inertia -->
+      </inertial>
+    </link>
+    <link name="${gripper_prefix}left_finger_tcp">
+      <inertial>
+        <origin rpy="0 0 0" xyz="0 0 0"/>
+        <mass value="0.01"/> <!-- Adjusted mass -->
+        <inertia ixx="0.00001" ixy="0" ixz="0" iyy="0.00001" iyz="0" izz="0.00001"/> <!-- Adjusted inertia -->
+      </inertial>
+    </link>
+    <link name="${gripper_prefix}right_finger_tcp">
+      <inertial>
+        <origin rpy="0 0 0" xyz="0 0 0"/>
+        <mass value="0.01"/> <!-- Adjusted mass -->
+        <inertia ixx="0.00001" ixy="0" ixz="0" iyy="0.00001" iyz="0" izz="0.00001"/> <!-- Adjusted inertia -->
+      </inertial>
+    </link>
+    <!-- Example joint with valid pose values -->
+    <joint name="${gripper_prefix}open_fingers_tcp_joint" type="fixed">
       <origin rpy="0 0 0" xyz="0 0 0.15"/>
-      <parent link="${prefix}base_link"/>
-      <child link="${prefix}tcp"/>
-      <axis xyz="0 0 1"/>
-    </joint>
-    <joint name="${prefix}closed_fingers_tcp_joint" type="fixed">
+      <parent link="${gripper_prefix}base_link"/>
+      <child link="${gripper_prefix}tcp"/>
+      <axis xyz="0 0 1"/>
+    </joint>
+    <joint name="${gripper_prefix}closed_fingers_tcp_joint" type="fixed">
       <origin rpy="0 0 0" xyz="0 0 0.20"/>
-      <parent link="${prefix}base_link"/>
-      <child link="${prefix}closed_fingers_tcp"/>
-      <axis xyz="0 0 1"/>
-    </joint>
-    <!-- left finger joints -->
-    <joint name="${prefix}left_outer_knuckle_joint" type="revolute">
+      <parent link="${gripper_prefix}base_link"/>
+      <child link="${gripper_prefix}closed_fingers_tcp"/>
+      <axis xyz="0 0 1"/>
+    </joint>
+    <!-- left finger joints with valid pose values and valid inertial values -->
+    <joint name="${gripper_prefix}left_outer_knuckle_joint" type="revolute">
       <origin rpy="0 0 0" xyz="0 -0.0325 0.0825"/>
-      <parent link="${prefix}base_link"/>
-      <child link="${prefix}left_outer_bar"/>
-      <axis xyz="1 0 0"/>
-      <limit effort="0" lower="-0.155" upper="0.7854" velocity="2.0"/>
-      <mimic joint="${prefix}finger_width_joint" multiplier="9.404" offset="-0.155"/>
-    </joint>
-    <joint name="${prefix}left_inner_knuckle_joint" type="revolute">
+      <parent link="${gripper_prefix}base_link"/>
+      <child link="${gripper_prefix}left_outer_bar"/>
+      <axis xyz="1 0 0"/>
+      <limit effort="0" lower="-0.155" upper="0.7854" velocity="2.0"/>
+      <mimic joint="${gripper_prefix}finger_width_joint" multiplier="9.404" offset="-0.155"/>
+    </joint>
+    <joint name="${gripper_prefix}left_inner_knuckle_joint" type="revolute">
       <origin rpy="0 0 0" xyz="0 -0.0165 0.0995"/>
-      <parent link="${prefix}base_link"/>
-      <child link="${prefix}left_inner_bar"/>
-      <axis xyz="1 0 0"/>
-      <limit effort="0" lower="-0.155" upper="0.7854" velocity="2.0"/>
-      <mimic joint="${prefix}left_outer_knuckle_joint" multiplier="1" offset="0"/>
-    </joint>
-    <joint name="${prefix}left_inner_finger_joint" type="revolute">
+      <parent link="${gripper_prefix}base_link"/>
+      <child link="${gripper_prefix}left_inner_bar"/>
+      <axis xyz="1 0 0"/>
+      <limit effort="0" lower="-0.155" upper="0.7854" velocity="2.0"/>
+      <mimic joint="${gripper_prefix}left_outer_knuckle_joint" multiplier="1" offset="0"/>
+    </joint>
+    <joint name="${gripper_prefix}left_inner_finger_joint" type="revolute">
       <origin rpy="0 0 0" xyz="0 0 0.058"/>
-      <parent link="${prefix}left_outer_bar"/>
-      <child link="${prefix}left_finger_mount"/>
+      <parent link="${gripper_prefix}left_outer_bar"/>
+      <child link="${gripper_prefix}left_finger_mount"/>
       <axis xyz="1 0 0"/>
       <limit effort="0" lower="-0.7854" upper="0.155" velocity="2.0"/>
-      <mimic joint="${prefix}left_outer_knuckle_joint" multiplier="-1" offset="0"/>
-    </joint>
-    <joint name="${prefix}left_inner_finger_pad_joint" type="fixed">
+      <mimic joint="${gripper_prefix}left_outer_knuckle_joint" multiplier="-1" offset="0"/>
+    </joint>
+    <joint name="${gripper_prefix}left_inner_finger_pad_joint" type="fixed">
       <origin rpy="0 0 0" xyz="0 0.010 0.0235"/>
-      <parent link="${prefix}left_finger_mount"/>
-      <child link="${prefix}left_finger_tip"/>
-      <axis xyz="0 0 1"/>
-    </joint>
-    <joint name="${prefix}left_finger_tcp_joint" type="fixed">
+      <parent link="${gripper_prefix}left_finger_mount"/>
+      <child link="${gripper_prefix}left_finger_tip"/>
+      <axis xyz="0 0 1"/>
+    </joint>
+    <joint name="${gripper_prefix}left_finger_tcp_joint" type="fixed">
       <origin rpy="0 0 0" xyz="0 0.0135 0.036"/>
-      <parent link="${prefix}left_finger_tip"/>
-      <child link="${prefix}left_finger_tcp"/>
-      <axis xyz="0 0 1"/>
-    </joint>
-    <!-- right finger joints -->
-    <joint name="${prefix}right_outer_knuckle_joint" type="revolute">
+      <parent link="${gripper_prefix}left_finger_tip"/>
+      <child link="${gripper_prefix}left_finger_tcp"/>
+      <axis xyz="0 0 1"/>
+    </joint>
+    <!-- right finger joints with valid pose values and valid inertial values -->
+    <joint name="${gripper_prefix}right_outer_knuckle_joint" type="revolute">
       <origin rpy="0 0 3.141592653589793" xyz="0 0.0325 0.0825"/>
-      <parent link="${prefix}base_link"/>
-      <child link="${prefix}right_outer_bar"/>
-      <axis xyz="1 0 0"/>
-      <limit effort="0" lower="-0.155" upper="0.7854" velocity="2.0"/>
-      <mimic joint="${prefix}left_outer_knuckle_joint" multiplier="1" offset="0"/>
-    </joint>
-    <joint name="${prefix}right_inner_knuckle_joint" type="revolute">
+      <parent link="${gripper_prefix}base_link"/>
+      <child link="${gripper_prefix}right_outer_bar"/>
+      <axis xyz="1 0 0"/>
+      <limit effort="0" lower="-0.155" upper="0.7854" velocity="2.0"/>
+      <mimic joint="${gripper_prefix}left_outer_knuckle_joint" multiplier="1" offset="0"/>
+    </joint>
+    <joint name="${gripper_prefix}right_inner_knuckle_joint" type="revolute">
       <origin rpy="0 0 3.141592653589793" xyz="0 0.0165 0.0995"/>
-      <parent link="${prefix}base_link"/>
-      <child link="${prefix}right_inner_bar"/>
-      <axis xyz="1 0 0"/>
-      <limit effort="0" lower="-0.155" upper="0.7854" velocity="2.0"/>
-      <mimic joint="${prefix}left_outer_knuckle_joint" multiplier="1" offset="0"/>
-    </joint>
-    <joint name="${prefix}right_inner_finger_joint" type="revolute">
+      <parent link="${gripper_prefix}base_link"/>
+      <child link="${gripper_prefix}right_inner_bar"/>
+      <axis xyz="1 0 0"/>
+      <limit effort="0" lower="-0.155" upper="0.7854" velocity="2.0"/>
+      <mimic joint="${gripper_prefix}left_outer_knuckle_joint" multiplier="1" offset="0"/>
+    </joint>
+    <joint name="${gripper_prefix}right_inner_finger_joint" type="revolute">
       <origin rpy="0 0 0" xyz="0 0 0.058"/>
-      <parent link="${prefix}right_outer_bar"/>
-      <child link="${prefix}right_finger_mount"/>
+      <parent link="${gripper_prefix}right_outer_bar"/>
+      <child link="${gripper_prefix}right_finger_mount"/>
       <axis xyz="1 0 0"/>
       <limit effort="0" lower="-0.7854" upper="0.155" velocity="2.0"/>
-      <mimic joint="${prefix}left_outer_knuckle_joint" multiplier="-1" offset="0"/>
-    </joint>
-    <joint name="${prefix}right_inner_finger_pad_joint" type="fixed">
+      <mimic joint="${gripper_prefix}left_outer_knuckle_joint" multiplier="-1" offset="0"/>
+    </joint>
+    <joint name="${gripper_prefix}right_inner_finger_pad_joint" type="fixed">
       <origin rpy="0 0 0" xyz="0 0.010 0.0235"/>
-      <parent link="${prefix}right_finger_mount"/>
-      <child link="${prefix}right_finger_tip"/>
-      <axis xyz="0 0 1"/>
-    </joint>
-    <joint name="${prefix}right_finger_tcp_joint" type="fixed">
+      <parent link="${gripper_prefix}right_finger_mount"/>
+      <child link="${gripper_prefix}right_finger_tip"/>
+      <axis xyz="0 0 1"/>
+    </joint>
+    <joint name="${gripper_prefix}right_finger_tcp_joint" type="fixed">
       <origin rpy="0 0 0" xyz="0 0.0135 0.036"/>
-      <parent link="${prefix}right_finger_tip"/>
-      <child link="${prefix}right_finger_tcp"/>
+      <parent link="${gripper_prefix}right_finger_tip"/>
+      <child link="${gripper_prefix}right_finger_tcp"/>
       <axis xyz="0 0 1"/>
     </joint>
     <!-- Control joint -->
-    <joint name="${prefix}finger_width_joint" type="revolute">
+    <joint name="${gripper_prefix}finger_width_joint" type="revolute">
       <origin rpy="0 0 0" xyz="0 0 0"/>
-      <parent link="${prefix}base_link"/>
-      <child link="${prefix}unused_finger_width_link"/>
+      <parent link="${gripper_prefix}base_link"/>
+      <child link="${gripper_prefix}unused_finger_width_link"/>
       <axis xyz="1 0 0"/>
       <limit effort="80" lower="0" upper="0.100" velocity="0.2"/>
     </joint>
-    <link name="${prefix}unused_finger_width_link">
-      <inertial>
-        <origin rpy="0 0 0" xyz="0 0 0"/>
-        <mass value="0.0001"/>
-        <inertia ixx="0.0000001" ixy="0" ixz="0" iyy="0.0000001" iyz="0" izz="0.0000001"/>
+    <link name="${gripper_prefix}unused_finger_width_link">
+      <inertial>
+        <origin rpy="0 0 0" xyz="0 0 0"/>
+        <mass value="0.01"/> <!-- Adjusted mass -->
+        <inertia ixx="0.00001" ixy="0" ixz="0" iyy="0.00001" iyz="0" izz="0.00001"/> <!-- Adjusted inertia -->
       </inertial>
     </link>

File: src/flexiv_ros2/flexiv_description/urdf/rizon.urdf.xacro (robot description, xacro)
@@ -10,5 +10,6 @@
   <xacro:include filename="$(find flexiv_description)/urdf/grav.urdf.xacro"/>
   <!-- parameters -->
-  <xacro:arg name="prefix" default="" />
+  <xacro:arg name="rizon_prefix" default="" />
+  <xacro:arg name="gripper_prefix" default="gripper_" />
   <xacro:arg name="robot_ip" default="" />
   <xacro:arg name="local_ip" default="" />
@@ -20,5 +21,5 @@
   <xacro:rizon_robot
     rizon_type="$(arg rizon_type)"
-    prefix="$(arg prefix)"
+    rizon_prefix="$(arg rizon_prefix)"
     robot_ip="$(arg robot_ip)"
     local_ip="$(arg local_ip)"
@@ -27,13 +28,11 @@
     initial_positions="${xacro.load_yaml(initial_positions_file)}">
   </xacro:rizon_robot>
-  <!-- Include the gripper macro with the appropriate prefix
-  <xacro:gripper prefix="$(arg prefix)"/>
-    <xacro:gripper prefix="gripper_"/>
-    <joint name="gripper_base_joint" type="fixed">
-      <origin xyz="0 0 0" rpy="0 0 0"/>
-      <parent link="flange"/>
-      <child link="gripper_base_link"/>
-    </joint>
-  -->
+  <!-- Include the gripper macro with the appropriate prefix-->
+  <xacro:gripper gripper_prefix="$(arg gripper_prefix)"/>
+  <joint name="$(arg gripper_prefix)base_joint" type="fixed">
+    <origin xyz="0 0 0" rpy="0 0 0"/>
+    <parent link="$(arg rizon_prefix)flange"/>
+    <child link="$(arg gripper_prefix)base_link"/>
+  </joint>
   <!-- JointStatePublisher publishes joint state information for the model.
          In future versions of Gazebo, replace 'ignition-gazebo' with 'gz-sim' and

File: src/flexiv_ros2/flexiv_description/urdf/rizon10.ros2_control.xacro (robot description, xacro)
@@ -2,5 +2,5 @@
 <robot xmlns:xacro="http://www.ros.org/wiki/xacro">
   <xacro:macro name="rizon10_ros2_control" params="
-    prefix
+    rizon_prefix
     robot_ip
     local_ip
@@ -22,5 +22,5 @@
         </xacro:unless>
       </hardware>
-      <joint name="${prefix}joint1">
+      <joint name="${rizon_prefix}joint1">
         <command_interface name="position">
           <param name="min">-2.7925</param>
@@ -39,5 +39,5 @@
         <state_interface name="effort"/>
       </joint>
-      <joint name="${prefix}joint2">
+      <joint name="${rizon_prefix}joint2">
         <command_interface name="position">
           <param name="min">-2.6704</param>
@@ -56,5 +56,5 @@
         <state_interface name="effort"/>
       </joint>
-      <joint name="${prefix}joint3">
+      <joint name="${rizon_prefix}joint3">
         <command_interface name="position">
           <param name="min">-2.7925</param>
@@ -73,5 +73,5 @@
         <state_interface name="effort"/>
       </joint>
-      <joint name="${prefix}joint4">
+      <joint name="${rizon_prefix}joint4">
         <command_interface name="position">
           <param name="min">-2.7053</param>
@@ -90,5 +90,5 @@
         <state_interface name="effort"/>
       </joint>
-      <joint name="${prefix}joint5">
+      <joint name="${rizon_prefix}joint5">
         <command_interface name="position">
           <param name="min">-2.9671</param>
@@ -107,5 +107,5 @@
         <state_interface name="effort"/>
       </joint>
-      <joint name="${prefix}joint6">
+      <joint name="${rizon_prefix}joint6">
         <command_interface name="position">
           <param name="min">-1.3963</param>
@@ -124,5 +124,5 @@
         <state_interface name="effort"/>
       </joint>
-      <joint name="${prefix}joint7">
+      <joint name="${rizon_prefix}joint7">
         <command_interface name="position">
           <param name="min">-2.9671</param>
@@ -141,5 +141,5 @@
         <state_interface name="effort"/>
       </joint>
-      <sensor name="${prefix}force_torque_sensor">
+      <sensor name="${rizon_prefix}force_torque_sensor">
         <state_interface name="force.x"/>
         <state_interface name="force.y"/>
@@ -149,5 +149,5 @@
         <state_interface name="torque.z"/>
       </sensor>
-      <sensor name="${prefix}external_wrench_in_base">
+      <sensor name="${rizon_prefix}external_wrench_in_base">
         <state_interface name="force.x"/>
         <state_interface name="force.y"/>
@@ -157,5 +157,5 @@
         <state_interface name="torque.z"/>
       </sensor>
-      <sensor name="${prefix}external_wrench_in_tcp">
+      <sensor name="${rizon_prefix}external_wrench_in_tcp">
         <state_interface name="force.x"/>
         <state_interface name="force.y"/>
@@ -165,5 +165,5 @@
         <state_interface name="torque.z"/>
       </sensor>
-      <sensor name="${prefix}tcp_pose">
+      <sensor name="${rizon_prefix}tcp_pose">
         <state_interface name="position.x"/>
         <state_interface name="position.y"/>
