Commit message: added gripper

File: src/flexiv_ros2/flexiv_description/urdf/rizon4.ros2_control.xacro (robot description, xacro)
@@ -2,5 +2,5 @@
 <robot xmlns:xacro="http://www.ros.org/wiki/xacro">
   <xacro:macro name="rizon4_ros2_control" params="
-    prefix
+    rizon_prefix
     robot_ip
     local_ip
@@ -20,8 +20,8 @@
           <param name="robot_ip">${robot_ip}</param>
           <param name="local_ip">${local_ip}</param>
-          <param name="prefix">${prefix}</param>
+          <param name="rizon_prefix">${rizon_prefix}</param>
         </xacro:unless>
       </hardware>
-      <joint name="${prefix}joint1">
+      <joint name="${rizon_prefix}joint1">
         <command_interface name="position">
           <param name="min">-2.7925</param>
@@ -40,5 +40,5 @@
         <state_interface name="effort"/>
       </joint>
-      <joint name="${prefix}joint2">
+      <joint name="${rizon_prefix}joint2">
         <command_interface name="position">
           <param name="min">-2.2689</param>
@@ -57,5 +57,5 @@
         <state_interface name="effort"/>
       </joint>
-      <joint name="${prefix}joint3">
+      <joint name="${rizon_prefix}joint3">
         <command_interface name="position">
           <param name="min">-2.9671</param>
@@ -74,5 +74,5 @@
         <state_interface name="effort"/>
       </joint>
-      <joint name="${prefix}joint4">
+      <joint name="${rizon_prefix}joint4">
         <command_interface name="position">
           <param name="min">-1.8675</param>
@@ -91,5 +91,5 @@
         <state_interface name="effort"/>
       </joint>
-      <joint name="${prefix}joint5">
+      <joint name="${rizon_prefix}joint5">
         <command_interface name="position">
           <param name="min">-2.9671</param>
@@ -108,5 +108,5 @@
         <state_interface name="effort"/>
       </joint>
-      <joint name="${prefix}joint6">
+      <joint name="${rizon_prefix}joint6">
         <command_interface name="position">
           <param name="min">-1.3963</param>
@@ -125,5 +125,5 @@
         <state_interface name="effort"/>
       </joint>
-      <joint name="${prefix}joint7">
+      <joint name="${rizon_prefix}joint7">
         <command_interface name="position">
           <param name="min">-2.9671</param>
@@ -142,5 +142,5 @@
         <state_interface name="effort"/>
       </joint>
-      <sensor name="${prefix}force_torque_sensor">
+      <sensor name="${rizon_prefix}force_torque_sensor">
         <state_interface name="force.x"/>
         <state_interface name="force.y"/>
@@ -150,5 +150,5 @@
         <state_interface name="torque.z"/>
       </sensor>
-      <sensor name="${prefix}external_wrench_in_base">
+      <sensor name="${rizon_prefix}external_wrench_in_base">
         <state_interface name="force.x"/>
         <state_interface name="force.y"/>
@@ -158,5 +158,5 @@
         <state_interface name="torque.z"/>
       </sensor>
-      <sensor name="${prefix}external_wrench_in_tcp">
+      <sensor name="${rizon_prefix}external_wrench_in_tcp">
         <state_interface name="force.x"/>
         <state_interface name="force.y"/>
@@ -166,5 +166,5 @@
         <state_interface name="torque.z"/>
       </sensor>
-      <sensor name="${prefix}tcp_pose">
+      <sensor name="${rizon_prefix}tcp_pose">
         <state_interface name="position.x"/>
         <state_interface name="position.y"/>
@@ -175,5 +175,5 @@
         <state_interface name="orientation.w"/>
       </sensor>
-      <gpio name="${prefix}gpio">
+      <gpio name="${rizon_prefix}gpio">
         <command_interface name="digital_output_0"/>
         <command_interface name="digital_output_1"/>

File: src/flexiv_ros2/flexiv_description/urdf/rizon4_joints_links.xacro (robot description, xacro)
@@ -3,67 +3,67 @@
   <!--
     rizon_type = "rizon4", "rizon4s"
-    prefix = "", "left_"
-    mesh_prefix_path = "", "package://flexiv_description/"
+    rizon_prefix = "", "left_"
+    mesh_rizon_prefix_path = "", "package://flexiv_description/"
     NOTE: accurate kinematic but approximated dynamics parameters
   -->
-  <xacro:macro name="rizon4_joints_links" params="rizon_type prefix mesh_prefix_path">
+  <xacro:macro name="rizon4_joints_links" params="rizon_type rizon_prefix mesh_rizon_prefix_path">
     <!-- JOINTS-->
-    <joint name="${prefix}base_joint" type="fixed">
+    <joint name="${rizon_prefix}base_joint" type="fixed">
       <parent link="world"/>
-      <child link="${prefix}base_link" />
+      <child link="${rizon_prefix}base_link" />
       <origin xyz="0.0 0.0 0.0" rpy="0.0 0.0 0.0"/>
     </joint>
-    <joint name="${prefix}joint1" type="revolute">
-      <parent link="${prefix}base_link"/>
-      <child link="${prefix}link1"/>
+    <joint name="${rizon_prefix}joint1" type="revolute">
+      <parent link="${rizon_prefix}base_link"/>
+      <child link="${rizon_prefix}link1"/>
       <origin xyz="0.0 0.0 0.155" rpy="0 0 ${-pi}"/>
       <axis xyz="0 0 1"/>
       <limit effort="123" lower="-2.7925" upper="2.7925" velocity="2.0944"/>
     </joint>
-    <joint name="${prefix}joint2" type="revolute">
-      <parent link="${prefix}link1"/>
-      <child link="${prefix}link2"/>
+    <joint name="${rizon_prefix}joint2" type="revolute">
+      <parent link="${rizon_prefix}link1"/>
+      <child link="${rizon_prefix}link2"/>
       <origin xyz="0.0 0.03 0.210" rpy="0 0 0"/>
       <axis xyz="0 1 0"/>
       <limit effort="123" lower="-2.2689" upper="2.2689" velocity="2.0944"/>
     </joint>
-    <joint name="${prefix}joint3" type="revolute">
-      <parent link="${prefix}link2"/>
-      <child link="${prefix}link3"/>
+    <joint name="${rizon_prefix}joint3" type="revolute">
+      <parent link="${rizon_prefix}link2"/>
+      <child link="${rizon_prefix}link3"/>
       <origin xyz="0.0 0.035 0.205" rpy="0 0 0"/>
       <axis xyz="0 0 1"/>
       <limit effort="64" lower="-2.9671" upper="2.9671" velocity="2.4435"/>
     </joint>
-    <joint name="${prefix}joint4" type="revolute">
-      <parent link="${prefix}link3"/>
-      <child link="${prefix}link4"/>
+    <joint name="${rizon_prefix}joint4" type="revolute">
+      <parent link="${rizon_prefix}link3"/>
+      <child link="${rizon_prefix}link4"/>
       <origin xyz="-0.02 -0.03 0.19" rpy="0 0 ${-pi}"/>
       <axis xyz="0 1 0"/>
       <limit effort="64" lower="-1.8675" upper="2.6878" velocity="2.4435" />
     </joint>
-    <joint name="${prefix}joint5" type="revolute">
-      <parent link="${prefix}link4"/>
-      <child link="${prefix}link5"/>
+    <joint name="${rizon_prefix}joint5" type="revolute">
+      <parent link="${rizon_prefix}link4"/>
+      <child link="${rizon_prefix}link5"/>
       <origin xyz="-0.02 0.025 0.195" rpy="0 0 ${-pi}"/>
       <axis xyz="0 0 1"/>
       <limit effort="39" lower="-2.9671" upper="2.9671" velocity="4.8869" />
     </joint>
-    <joint name="${prefix}joint6" type="revolute">
-      <parent link="${prefix}link5"/>
-      <child link="${prefix}link6"/>
+    <joint name="${rizon_prefix}joint6" type="revolute">
+      <parent link="${rizon_prefix}link5"/>
+      <child link="${rizon_prefix}link6"/>
       <origin xyz="0.0 0.03 0.19" rpy="0 0 0"/>
       <axis xyz="0 1 0"/>
       <limit effort="39" lower="-1.3963" upper="4.5379" velocity="4.8869" />
     </joint>
-    <joint name="${prefix}joint7" type="revolute">
-      <parent link="${prefix}link6"/>
-      <child link="${prefix}link7"/>
+    <joint name="${rizon_prefix}joint7" type="revolute">
+      <parent link="${rizon_prefix}link6"/>
+      <child link="${rizon_prefix}link7"/>
       <origin xyz="-0.055 0.070 0.11" rpy="0 ${-pi/2} 0"/>
       <axis xyz="0 0 1"/>
       <limit effort="39" lower="-2.9671" upper="2.9671" velocity="4.8869" />
     </joint>
-    <joint name="${prefix}link7_to_flange" type="fixed">
-      <parent link="${prefix}link7"/>
-      <child link="${prefix}flange"/>
+    <joint name="${rizon_prefix}link7_to_flange" type="fixed">
+      <parent link="${rizon_prefix}link7"/>
+      <child link="${rizon_prefix}flange"/>
       <xacro:if value="${rizon_type=='rizon4'}">
         <origin xyz="0.0 0.0 0.081" rpy="0 0 ${-pi}"/>
@@ -76,5 +76,5 @@
     <link name="world">
     </link>
-    <link name="${prefix}base_link">
+    <link name="${rizon_prefix}base_link">
       <inertial>
         <mass value="3.7" />
@@ -85,16 +85,16 @@
         <origin xyz="0 0 0" rpy="0 0 0"/>
         <geometry>
-          <mesh filename="${mesh_prefix_path}meshes/${rizon_type}/visual/link0.obj" />
-        </geometry>
-        <material name="rizon_light_grey" />
-      </visual>
-      <collision>
-        <origin xyz="0 0 0" rpy="0 0 0"/>
-        <geometry>
-          <mesh filename="${mesh_prefix_path}meshes/${rizon_type}/collision/link0.stl" />
-        </geometry>
-      </collision>
-    </link>
-    <link name="${prefix}link1">
+          <mesh filename="${mesh_rizon_prefix_path}meshes/${rizon_type}/visual/link0.obj" />
+        </geometry>
+        <material name="rizon_light_grey" />
+      </visual>
+      <collision>
+        <origin xyz="0 0 0" rpy="0 0 0"/>
+        <geometry>
+          <mesh filename="${mesh_rizon_prefix_path}meshes/${rizon_type}/collision/link0.stl" />
+        </geometry>
+      </collision>
+    </link>
+    <link name="${rizon_prefix}link1">
       <inertial>
         <mass value="3.7" />
@@ -105,16 +105,16 @@
         <origin xyz="0 0 0" rpy="0 0 0" />
         <geometry>
-          <mesh filename="${mesh_prefix_path}meshes/${rizon_type}/visual/link1.obj" />
-        </geometry>
-        <material name="rizon_light_grey" />
-      </visual>
-      <collision>
-        <origin xyz="0 0 0" rpy="0 0 0" />
-        <geometry>
-          <mesh filename="${mesh_prefix_path}meshes/${rizon_type}/collision/link1.stl" />
-        </geometry>
-      </collision>
-    </link>
-    <link name="${prefix}link2">
+          <mesh filename="${mesh_rizon_prefix_path}meshes/${rizon_type}/visual/link1.obj" />
+        </geometry>
+        <material name="rizon_light_grey" />
+      </visual>
+      <collision>
+        <origin xyz="0 0 0" rpy="0 0 0" />
+        <geometry>
+          <mesh filename="${mesh_rizon_prefix_path}meshes/${rizon_type}/collision/link1.stl" />
+        </geometry>
+      </collision>
+    </link>
+    <link name="${rizon_prefix}link2">
       <inertial>
         <mass value="2.7" />
@@ -125,16 +125,16 @@
         <origin xyz="0 0 0" rpy="0 0 0"/>
         <geometry>
-          <mesh filename="${mesh_prefix_path}meshes/${rizon_type}/visual/link2.obj" />
-        </geometry>
-        <material name="rizon_light_grey" />
-      </visual>
-      <collision>
-        <origin xyz="0 0 0" rpy="0 0 0"/>
-        <geometry>
-          <mesh filename="${mesh_prefix_path}meshes/${rizon_type}/collision/link2.stl" />
-        </geometry>
-      </collision>
-    </link>
-    <link name="${prefix}link3">
+          <mesh filename="${mesh_rizon_prefix_path}meshes/${rizon_type}/visual/link2.obj" />
+        </geometry>
+        <material name="rizon_light_grey" />
+      </visual>
+      <collision>
+        <origin xyz="0 0 0" rpy="0 0 0"/>
+        <geometry>
+          <mesh filename="${mesh_rizon_prefix_path}meshes/${rizon_type}/collision/link2.stl" />
+        </geometry>
+      </collision>
+    </link>
+    <link name="${rizon_prefix}link3">
       <inertial>
         <mass value="2.4" />
@@ -145,16 +145,16 @@
         <origin xyz="0 0 0" rpy="0 0 0" />
         <geometry>
-          <mesh filename="${mesh_prefix_path}meshes/${rizon_type}/visual/link3.obj" />
-        </geometry>
-        <material name="rizon_light_grey" />
-      </visual>
-      <collision>
-        <origin xyz="0 0 0" rpy="0 0 0" />
-        <geometry>
-          <mesh filename="${mesh_prefix_path}meshes/${rizon_type}/collision/link3.stl" />
-        </geometry>
-      </collision>
-    </link>
-    <link name="${prefix}link4">
+          <mesh filename="${mesh_rizon_prefix_path}meshes/${rizon_type}/visual/link3.obj" />
+        </geometry>
+        <material name="rizon_light_grey" />
+      </visual>
+      <collision>
+        <origin xyz="0 0 0" rpy="0 0 0" />
+        <geometry>
+          <mesh filename="${mesh_rizon_prefix_path}meshes/${rizon_type}/collision/link3.stl" />
+        </geometry>
+      </collision>
+    </link>
+    <link name="${rizon_prefix}link4">
       <inertial>
         <mass value="2.4" />
@@ -165,16 +165,16 @@
         <origin xyz="0 0 0" rpy="0 0 0"/>
         <geometry>
-          <mesh filename="${mesh_prefix_path}meshes/${rizon_type}/visual/link4.obj" />
-        </geometry>
-        <material name="rizon_light_grey" />
-      </visual>
-      <collision>
-        <origin xyz="0 0 0" rpy="0 0 0"/>
-        <geometry>
-          <mesh filename="${mesh_prefix_path}meshes/${rizon_type}/collision/link4.stl" />
-        </geometry>
-      </collision>
-    </link>
-    <link name="${prefix}link5">
+          <mesh filename="${mesh_rizon_prefix_path}meshes/${rizon_type}/visual/link4.obj" />
+        </geometry>
+        <material name="rizon_light_grey" />
+      </visual>
+      <collision>
+        <origin xyz="0 0 0" rpy="0 0 0"/>
+        <geometry>
+          <mesh filename="${mesh_rizon_prefix_path}meshes/${rizon_type}/collision/link4.stl" />
+        </geometry>
+      </collision>
+    </link>
+    <link name="${rizon_prefix}link5">
       <inertial>
         <mass value="2.4" />
@@ -185,16 +185,16 @@
         <origin xyz="0 0 0" rpy="0 0 0"/>
         <geometry>
-          <mesh filename="${mesh_prefix_path}meshes/${rizon_type}/visual/link5.obj" />
-        </geometry>
-        <material name="rizon_light_grey" />
-      </visual>
-      <collision>
-        <origin xyz="0 0 0" rpy="0 0 0"/>
-        <geometry>
-          <mesh filename="${mesh_prefix_path}meshes/${rizon_type}/collision/link5.stl" />
-        </geometry>
-      </collision>
-    </link>
-    <link name="${prefix}link6">
+          <mesh filename="${mesh_rizon_prefix_path}meshes/${rizon_type}/visual/link5.obj" />
+        </geometry>
+        <material name="rizon_light_grey" />
+      </visual>
+      <collision>
+        <origin xyz="0 0 0" rpy="0 0 0"/>
+        <geometry>
+          <mesh filename="${mesh_rizon_prefix_path}meshes/${rizon_type}/collision/link5.stl" />
+        </geometry>
+      </collision>
+    </link>
+    <link name="${rizon_prefix}link6">
       <inertial>
         <mass value="2.1" />
@@ -205,16 +205,16 @@
         <origin xyz="0 0 0" rpy="0 0 0"/>
         <geometry>
-          <mesh filename="${mesh_prefix_path}meshes/${rizon_type}/visual/link6.obj" />
-        </geometry>
-        <material name="rizon_light_grey" />
-      </visual>
-      <collision>
-        <origin xyz="0 0 0" rpy="0 0 0"/>
-        <geometry>
-          <mesh filename="${mesh_prefix_path}meshes/${rizon_type}/collision/link6.stl" />
-        </geometry>
-      </collision>
-    </link>
-    <link name="${prefix}link7">
+          <mesh filename="${mesh_rizon_prefix_path}meshes/${rizon_type}/visual/link6.obj" />
+        </geometry>
+        <material name="rizon_light_grey" />
+      </visual>
+      <collision>
+        <origin xyz="0 0 0" rpy="0 0 0"/>
+        <geometry>
+          <mesh filename="${mesh_rizon_prefix_path}meshes/${rizon_type}/collision/link6.stl" />
+        </geometry>
+      </collision>
+    </link>
+    <link name="${rizon_prefix}link7">
       <xacro:if value="${rizon_type=='rizon4'}">
         <inertial>
@@ -226,5 +226,5 @@
           <origin xyz="0 0 0" rpy="0 0 0"/>
           <geometry>
-            <mesh filename="${mesh_prefix_path}meshes/${rizon_type}/visual/link7.obj" />
+            <mesh filename="${mesh_rizon_prefix_path}meshes/${rizon_type}/visual/link7.obj" />
           </geometry>
           <material name="rizon_light_grey" />
@@ -233,5 +233,5 @@
           <origin xyz="0 0 0" rpy="0 0 0"/>
           <geometry>
-            <mesh filename="${mesh_prefix_path}meshes/${rizon_type}/collision/link7.stl" />
+            <mesh filename="${mesh_rizon_prefix_path}meshes/${rizon_type}/collision/link7.stl" />
           </geometry>
         </collision>
@@ -246,5 +246,5 @@
           <origin xyz="0 0 0" rpy="0 0 0"/>
           <geometry>
-            <mesh filename="${mesh_prefix_path}meshes/${rizon_type}/visual/link7.obj" />
+            <mesh filename="${mesh_rizon_prefix_path}meshes/${rizon_type}/visual/link7.obj" />
           </geometry>
           <material name="rizon_light_grey" />
@@ -253,10 +253,10 @@
           <origin xyz="0 0 0" rpy="0 0 0"/>
           <geometry>
-            <mesh filename="${mesh_prefix_path}meshes/${rizon_type}/collision/link7.stl" />
+            <mesh filename="${mesh_rizon_prefix_path}meshes/${rizon_type}/collision/link7.stl" />
           </geometry>
         </collision>
       </xacro:if>
     </link>
-    <link name="${prefix}flange"/>
+    <link name="${rizon_prefix}flange"/>
   </xacro:macro>
 </robot>

File: src/flexiv_ros2/flexiv_description/urdf/rizon_macro.xacro (robot description, xacro)
@@ -3,5 +3,5 @@
   <xacro:macro name="rizon_robot" params="
     rizon_type
-    prefix
+    rizon_prefix
     robot_ip
     local_ip
@@ -15,8 +15,8 @@
     <xacro:if value="${rizon_type=='rizon4' or rizon_type=='rizon4s'}">
       <xacro:include filename="$(find flexiv_description)/urdf/rizon4_joints_links.xacro" />
-      <xacro:rizon4_joints_links rizon_type="${rizon_type}" prefix="${prefix}" mesh_prefix_path="package://flexiv_description/" />
+      <xacro:rizon4_joints_links rizon_type="${rizon_type}" rizon_prefix="${rizon_prefix}" mesh_rizon_prefix_path="package://flexiv_description/" />
       <!-- ros2 control include -->
       <xacro:include filename="$(find flexiv_description)/urdf/rizon4.ros2_control.xacro"/>
-      <xacro:rizon4_ros2_control prefix="${prefix}" robot_ip="${robot_ip}"
+      <xacro:rizon4_ros2_control rizon_prefix="${rizon_prefix}" robot_ip="${robot_ip}"
         local_ip="${local_ip}" use_fake_hardware="${use_fake_hardware}"
         fake_sensor_commands="${fake_sensor_commands}"
@@ -27,8 +27,8 @@
     <xacro:if value="${rizon_type=='rizon10'}">
       <xacro:include filename="$(find flexiv_description)/urdf/rizon10_joints_links.xacro" />
-      <xacro:rizon10_joints_links rizon_type="${rizon_type}" prefix="${prefix}" mesh_prefix_path="package://flexiv_description/" />
+      <xacro:rizon10_joints_links rizon_type="${rizon_type}" rizon_prefix="${rizon_prefix}" mesh_rizon_prefix_path="package://flexiv_description/" />
       <!-- ros2 control include -->
       <xacro:include filename="$(find flexiv_description)/urdf/rizon10.ros2_control.xacro"/>
-      <xacro:rizon10_ros2_control prefix="${prefix}" robot_ip="${robot_ip}"
+      <xacro:rizon10_ros2_control rizon_prefix="${rizon_prefix}" robot_ip="${robot_ip}"
         local_ip="${local_ip}" use_fake_hardware="${use_fake_hardware}"
         fake_sensor_commands="${fake_sensor_commands}"
