Commit message: time synced, need to publish gripper joints to joint_states

File: src/flexiv_ros2/flexiv_description/urdf/grav.urdf.xacro (robot description, xacro)
@@ -27,6 +27,6 @@
       <inertial>
         <origin xyz="0 0 0.029" rpy="0 0 0"/>
-        <mass value="0.01"/> <!-- Adjusted mass -->
-        <inertia ixx="0.00001" ixy="0" ixz="0" iyy="0.00001" iyz="0" izz="0.00001"/> <!-- Adjusted inertia -->
+        <mass value="0.0001"/>
+        <inertia ixx="0.0000001" ixy="0" ixz="0" iyy="0.0000001" iyz="0" izz="0.0000001"/>
       </inertial>
       <visual>
@@ -41,6 +41,6 @@
       <inertial>
         <origin xyz="0 0 0.029" rpy="0 0 0"/>
-        <mass value="0.01"/> <!-- Adjusted mass -->
-        <inertia ixx="0.00001" ixy="0" ixz="0" iyy="0.00001" iyz="0" izz="0.00001"/> <!-- Adjusted inertia -->
+        <mass value="0.0001"/>
+        <inertia ixx="0.0000001" ixy="0" ixz="0" iyy="0.0000001" iyz="0" izz="0.0000001"/>
       </inertial>
       <visual>
@@ -56,6 +56,6 @@
       <inertial>
         <origin xyz="0 0 0" rpy="0 0 0"/>
-        <mass value="0.01"/> <!-- Adjusted mass -->
-        <inertia ixx="0.00001" ixy="0" ixz="0" iyy="0.00001" iyz="0" izz="0.00001"/> <!-- Adjusted inertia -->
+        <mass value="0.0001"/>
+        <inertia ixx="0.0000001" ixy="0" ixz="0" iyy="0.0000001" iyz="0" izz="0.0000001"/>
       </inertial>
       <visual>
@@ -70,6 +70,6 @@
       <inertial>
         <origin rpy="0 0 0" xyz="0 0 0"/>
-        <mass value="0.01"/> <!-- Adjusted mass -->
-        <inertia ixx="0.00001" ixy="0" ixz="0" iyy="0.00001" iyz="0" izz="0.00001"/> <!-- Adjusted inertia -->
+        <mass value="0.0001"/>
+        <inertia ixx="0.0000001" ixy="0" ixz="0" iyy="0.0000001" iyz="0" izz="0.0000001"/>
       </inertial>
       <visual>
@@ -90,6 +90,6 @@
       <inertial>
         <origin xyz="0 0 0.029" rpy="0 0 0"/>
-        <mass value="0.01"/> <!-- Adjusted mass -->
-        <inertia ixx="0.00001" ixy="0" ixz="0" iyy="0.00001" iyz="0" izz="0.00001"/> <!-- Adjusted inertia -->
+        <mass value="0.0001"/>
+        <inertia ixx="0.0000001" ixy="0" ixz="0" iyy="0.0000001" iyz="0" izz="0.0000001"/>
       </inertial>
       <visual>
@@ -104,6 +104,6 @@
       <inertial>
         <origin xyz="0 0 0.029" rpy="0 0 0"/>
-        <mass value="0.01"/> <!-- Adjusted mass -->
-        <inertia ixx="0.00001" ixy="0" ixz="0" iyy="0.00001" iyz="0" izz="0.00001"/> <!-- Adjusted inertia -->
+        <mass value="0.0001"/>
+        <inertia ixx="0.0000001" ixy="0" ixz="0" iyy="0.0000001" iyz="0" izz="0.0000001"/>
       </inertial>
       <visual>
@@ -118,6 +118,6 @@
       <inertial>
         <origin xyz="0 0 0" rpy="0 0 0"/>
-        <mass value="0.01"/> <!-- Adjusted mass -->
-        <inertia ixx="0.00001" ixy="0" ixz="0" iyy="0.00001" iyz="0" izz="0.00001"/> <!-- Adjusted inertia -->
+        <mass value="0.0001"/>
+        <inertia ixx="0.0000001" ixy="0" ixz="0" iyy="0.0000001" iyz="0" izz="0.0000001"/>
       </inertial>
       <visual>
@@ -132,6 +132,6 @@
       <inertial>
         <origin rpy="0 0 0" xyz="0 0 0"/>
-        <mass value="0.01"/> <!-- Adjusted mass -->
-        <inertia ixx="0.00001" ixy="0" ixz="0" iyy="0.00001" iyz="0" izz="0.00001"/> <!-- Adjusted inertia -->
+        <mass value="0.0001"/>
+        <inertia ixx="0.0000001" ixy="0" ixz="0" iyy="0.0000001" iyz="0" izz="0.0000001"/>
       </inertial>
       <visual>
@@ -152,6 +152,6 @@
       <inertial>
         <origin rpy="0 0 0" xyz="0 0 0"/>
-        <mass value="0.01"/> <!-- Adjusted mass -->
-        <inertia ixx="0.00001" ixy="0" ixz="0" iyy="0.00001" iyz="0" izz="0.00001"/> <!-- Adjusted inertia -->
+        <mass value="0"/>
+        <inertia ixx="0" ixy="0" ixz="0" iyy="0" iyz="0" izz="0"/>
       </inertial>
     </link>
@@ -159,6 +159,6 @@
       <inertial>
         <origin rpy="0 0 0" xyz="0 0 0"/>
-        <mass value="0.01"/> <!-- Adjusted mass -->
-        <inertia ixx="0.00001" ixy="0" ixz="0" iyy="0.00001" iyz="0" izz="0.00001"/> <!-- Adjusted inertia -->
+        <mass value="0"/>
+        <inertia ixx="0" ixy="0" ixz="0" iyy="0" iyz="0" izz="0"/>
       </inertial>
     </link>
@@ -166,6 +166,6 @@
       <inertial>
         <origin rpy="0 0 0" xyz="0 0 0"/>
-        <mass value="0.01"/> <!-- Adjusted mass -->
-        <inertia ixx="0.00001" ixy="0" ixz="0" iyy="0.00001" iyz="0" izz="0.00001"/> <!-- Adjusted inertia -->
+        <mass value="0"/>
+        <inertia ixx="0" ixy="0" ixz="0" iyy="0" iyz="0" izz="0"/>
       </inertial>
     </link>
@@ -173,6 +173,6 @@
       <inertial>
         <origin rpy="0 0 0" xyz="0 0 0"/>
-        <mass value="0.01"/> <!-- Adjusted mass -->
-        <inertia ixx="0.00001" ixy="0" ixz="0" iyy="0.00001" iyz="0" izz="0.00001"/> <!-- Adjusted inertia -->
+        <mass value="0"/>
+        <inertia ixx="0" ixy="0" ixz="0" iyy="0" iyz="0" izz="0"/>
       </inertial>
     </link>

File: src/flexiv_ros2/flexiv_description/urdf/rizon.urdf.xacro (robot description, xacro)
@@ -4,5 +4,5 @@
   <xacro:arg name="name" default="rizon"/>
   <!-- 'rizon_type' values: rizon4, rizon4s, rizon10 -->
-  <xacro:arg name="rizon_type" default="rizon4"/>
+  <xacro:arg name="rizon_type" default="rizon4s"/>
   <!-- import main macro -->
   <xacro:include filename="$(find flexiv_description)/urdf/rizon_macro.xacro"/>

File: src/flexiv_ros2/flexiv_description/urdf/rizon_macro.xacro (robot description, xacro)
@@ -1,4 +1,4 @@
 <?xml version="1.0"?>
-<robot xmlns:xacro="http://wiki.ros.org/xacro">
+<robot xmlns:xacro="http://www.ros.org/wiki/xacro">
   <xacro:macro name="rizon_robot" params="
     rizon_type

Commit message: fixed joints fixed tf issue

File: src/flexiv_ros2/flexiv_description/urdf/grav.urdf.xacro (robot description, xacro)
@@ -148,5 +148,5 @@
       </collision>
     </link>
-    <!-- TCP links -->
+    <!-- TCP links
     <link name="${gripper_prefix}tcp">
       <inertial>
@@ -177,5 +177,6 @@
       </inertial>
     </link>
-    <!-- Example joint with valid pose values -->
+    -->
+    <!-- Example joint with valid pose values
     <joint name="${gripper_prefix}open_fingers_tcp_joint" type="fixed">
       <origin rpy="0 0 0" xyz="0 0 0.15"/>
@@ -190,6 +191,7 @@
       <axis xyz="0 0 1"/>
     </joint>
+    -->
     <!-- left finger joints with valid pose values and valid inertial values -->
-    <joint name="${gripper_prefix}left_outer_knuckle_joint" type="revolute">
+    <joint name="${gripper_prefix}left_outer_knuckle_joint" type="fixed">
       <origin rpy="0 0 0" xyz="0 -0.0325 0.0825"/>
       <parent link="${gripper_prefix}base_link"/>
@@ -199,5 +201,5 @@
       <mimic joint="${gripper_prefix}finger_width_joint" multiplier="9.404" offset="-0.155"/>
     </joint>
-    <joint name="${gripper_prefix}left_inner_knuckle_joint" type="revolute">
+    <joint name="${gripper_prefix}left_inner_knuckle_joint" type="fixed">
       <origin rpy="0 0 0" xyz="0 -0.0165 0.0995"/>
       <parent link="${gripper_prefix}base_link"/>
@@ -207,5 +209,5 @@
       <mimic joint="${gripper_prefix}left_outer_knuckle_joint" multiplier="1" offset="0"/>
     </joint>
-    <joint name="${gripper_prefix}left_inner_finger_joint" type="revolute">
+    <joint name="${gripper_prefix}left_inner_finger_joint" type="fixed">
       <origin rpy="0 0 0" xyz="0 0 0.058"/>
       <parent link="${gripper_prefix}left_outer_bar"/>
@@ -221,4 +223,5 @@
       <axis xyz="0 0 1"/>
     </joint>
+    <!--
     <joint name="${gripper_prefix}left_finger_tcp_joint" type="fixed">
       <origin rpy="0 0 0" xyz="0 0.0135 0.036"/>
@@ -227,6 +230,7 @@
       <axis xyz="0 0 1"/>
     </joint>
+    -->
     <!-- right finger joints with valid pose values and valid inertial values -->
-    <joint name="${gripper_prefix}right_outer_knuckle_joint" type="revolute">
+    <joint name="${gripper_prefix}right_outer_knuckle_joint" type="fixed">
       <origin rpy="0 0 3.141592653589793" xyz="0 0.0325 0.0825"/>
       <parent link="${gripper_prefix}base_link"/>
@@ -236,5 +240,5 @@
       <mimic joint="${gripper_prefix}left_outer_knuckle_joint" multiplier="1" offset="0"/>
     </joint>
-    <joint name="${gripper_prefix}right_inner_knuckle_joint" type="revolute">
+    <joint name="${gripper_prefix}right_inner_knuckle_joint" type="fixed">
       <origin rpy="0 0 3.141592653589793" xyz="0 0.0165 0.0995"/>
       <parent link="${gripper_prefix}base_link"/>
@@ -244,5 +248,5 @@
       <mimic joint="${gripper_prefix}left_outer_knuckle_joint" multiplier="1" offset="0"/>
     </joint>
-    <joint name="${gripper_prefix}right_inner_finger_joint" type="revolute">
+    <joint name="${gripper_prefix}right_inner_finger_joint" type="fixed">
       <origin rpy="0 0 0" xyz="0 0 0.058"/>
       <parent link="${gripper_prefix}right_outer_bar"/>
@@ -258,4 +262,5 @@
       <axis xyz="0 0 1"/>
     </joint>
+    <!--
     <joint name="${gripper_prefix}right_finger_tcp_joint" type="fixed">
       <origin rpy="0 0 0" xyz="0 0.0135 0.036"/>
@@ -264,6 +269,7 @@
       <axis xyz="0 0 1"/>
     </joint>
+    -->
     <!-- Control joint -->
-    <joint name="${gripper_prefix}finger_width_joint" type="revolute">
+    <joint name="${gripper_prefix}finger_width_joint" type="fixed">
       <origin rpy="0 0 0" xyz="0 0 0"/>
       <parent link="${gripper_prefix}base_link"/>
@@ -275,6 +281,6 @@
       <inertial>
         <origin rpy="0 0 0" xyz="0 0 0"/>
-        <mass value="0.01"/> <!-- Adjusted mass -->
-        <inertia ixx="0.00001" ixy="0" ixz="0" iyy="0.00001" iyz="0" izz="0.00001"/> <!-- Adjusted inertia -->
+        <mass value="0.0001"/>
+        <inertia ixx="0.0000001" ixy="0" ixz="0" iyy="0.0000001" iyz="0" izz="0.0000001"/>
       </inertial>
     </link>
